File: rectificacion/rectificador.brd (EAGLE design)
At the start: 9 parts

Commit message: Regulator ready to get gerbers
Parts:
- added IC1: (no value), v-reg:317TS
- added R1: (no value), rcl:0204/7
- added R2: (no value), rcl:RTRIM64W
- moved C1 6.35 mm to (19.1, 24.1)
- moved X3 5.08 mm to (40.6, 22.9)
Connections:
- new net N$1: IC1.1, R1.1, R2.3
- new net OUT: IC1.2, R1.2, X3.1
- net GND: now also R2.2
- net VCC: now also IC1.3; no longer X3.1
Routing:
- net OUT: track 0.00 -> 17.4 mm
- net N$1: track 0.00 -> 14.3 mm
- net VCC: track 33.6 -> 23.7 mm
