File: rectificacion/rectificador.sch (EAGLE design)
At the start: 9 parts

Commit message: Regulator ready to get gerbers
Parts:
- added IC1: (no value), v-reg:LM317TS
- added R1: (no value), rcl:R-US_0204/7
- added R2: (no value), rcl:R-TRIMM64W
Connections:
- new net N$1: IC1.ADJ, R1.1, R2.E
- new net OUT: IC1.OUT, R1.2, X3-1.KL
- net GND: now also R2.S
- net VCC: now also IC1.IN; no longer X3-1.KL
Other:
- moved on the sheet: C1
Changed lines of the file:
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@@
 <part name="SUPPLY3" library="supply2" library_urn="urn:adsk.eagle:library:372" deviceset="GND" device=""/>
 <part name="SUPPLY4" library="supply2" library_urn="urn:adsk.eagle:library:372" deviceset="GND" device=""/>
+<part name="IC1" library="v-reg" library_urn="urn:adsk.eagle:library:409" deviceset="LM317TS" device="" package3d_urn="urn:adsk.eagle:package:30353/1"/>
+<part name="R1" library="rcl" library_urn="urn:adsk.eagle:library:334" deviceset="R-US_" device="0204/7" package3d_urn="urn:adsk.eagle:package:23498/2"/>
+<part name="R2" library="rcl" library_urn="urn:adsk.eagle:library:334" deviceset="R-TRIMM" device="64W" package3d_urn="urn:adsk.eagle:package:23748/1"/>
+<part name="SUPPLY1" library="supply2" library_urn="urn:adsk.eagle:library:372" deviceset="GND" device=""/>
 </parts>
 <sheets>
@@
 <attribute name="VALUE" x="55.118" y="92.583" size="1.778" layer="96" rot="R270"/>
 </instance>
-<instance part="C1" gate="G$1" x="71.12" y="76.2" smashed="yes">
-<attribute name="NAME" x="72.136" y="76.835" size="1.778" layer="95"/>
-<attribute name="VALUE" x="72.136" y="72.009" size="1.778" layer="96"/>
+<instance part="C1" gate="G$1" x="66.04" y="86.36" smashed="yes">
+<attribute name="NAME" x="67.056" y="86.995" size="1.778" layer="95"/>
+<attribute name="VALUE" x="67.056" y="82.169" size="1.778" layer="96"/>
 </instance>
 <instance part="X3" gate="-1" x="12.7" y="53.34" smashed="yes">
@@
 <attribute name="VALUE" x="26.035" y="46.355" size="1.778" layer="96" rot="R90"/>
 </instance>
-<instance part="SUPPLY3" gate="GND" x="71.12" y="66.04" smashed="yes">
-<attribute name="VALUE" x="69.215" y="62.865" size="1.778" layer="96"/>
+<instance part="SUPPLY3" gate="GND" x="66.04" y="76.2" smashed="yes">
+<attribute name="VALUE" x="64.135" y="73.025" size="1.778" layer="96"/>
 </instance>
 <instance part="SUPPLY4" gate="GND" x="58.42" y="83.82" smashed="yes">
 <attribute name="VALUE" x="56.515" y="80.645" size="1.778" layer="96"/>
+</instance>
+<instance part="IC1" gate="1" x="50.8" y="45.72" smashed="yes">
+<attribute name="NAME" x="53.34" y="38.1" size="1.778" layer="95"/>
+<attribute name="VALUE" x="53.34" y="35.56" size="1.778" layer="96"/>
+</instance>
+<instance part="R1" gate="G$1" x="60.96" y="38.1" smashed="yes" rot="R90">
+<attribute name="NAME" x="59.4614" y="34.29" size="1.778" layer="95" rot="R90"/>
+<attribute name="VALUE" x="64.262" y="34.29" size="1.778" layer="96" rot="R90"/>
+</instance>
+<instance part="R2" gate="G$1" x="50.8" y="27.94" smashed="yes">
+<attribute name="NAME" x="44.831" y="24.13" size="1.778" layer="95" rot="R90"/>
+<attribute name="VALUE" x="46.99" y="24.13" size="1.778" layer="96" rot="R90"/>
+</instance>
+<instance part="SUPPLY1" gate="GND" x="58.42" y="22.86" smashed="yes">
+<attribute name="VALUE" x="56.515" y="19.685" size="1.778" layer="96"/>
 </instance>
 </instances>
@@
 <segment>
 <pinref part="C1" gate="G$1" pin="2"/>
-<wire x1="71.12" y1="71.12" x2="71.12" y2="68.58" width="0.1524" layer="91"/>
+<wire x1="66.04" y1="81.28" x2="66.04" y2="78.74" width="0.1524" layer="91"/>
 <pinref part="SUPPLY3" gate="GND" pin="GND"/>
 </segment>
@@
 <pinref part="SUPPLY4" gate="GND" pin="GND"/>
 </segment>
+<segment>
+<pinref part="R2" gate="G$1" pin="S"/>
+<wire x1="55.88" y1="27.94" x2="58.42" y2="27.94" width="0.1524" layer="91"/>
+<wire x1="58.42" y1="27.94" x2="58.42" y2="25.4" width="0.1524" layer="91"/>
+<pinref part="SUPPLY1" gate="GND" pin="GND"/>
+</segment>
 </net>
 <net name="6" class="0">
@@
 <segment>
 <pinref part="C1" gate="G$1" pin="1"/>
-<wire x1="71.12" y1="78.74" x2="71.12" y2="81.28" width="0.1524" layer="91"/>
-<label x="71.12" y="81.28" size="1.778" layer="95" xref="yes"/>
-</segment>
-<segment>
-<pinref part="X3" gate="-1" pin="KL"/>
-<wire x1="17.78" y1="53.34" x2="20.32" y2="53.34" width="0.1524" layer="91"/>
-<label x="20.32" y="53.34" size="1.778" layer="95" xref="yes"/>
+<wire x1="66.04" y1="88.9" x2="66.04" y2="91.44" width="0.1524" layer="91"/>
+<label x="66.04" y="91.44" size="1.778" layer="95" xref="yes"/>
+</segment>
+<segment>
+<pinref part="IC1" gate="1" pin="IN"/>
+<wire x1="43.18" y1="45.72" x2="40.64" y2="45.72" width="0.1524" layer="91"/>
+<label x="40.64" y="45.72" size="1.778" layer="95" rot="R180" xref="yes"/>
 </segment>
 </net>
@@
 </segment>
 </net>
+<net name="OUT" class="0">
+<segment>
+<pinref part="IC1" gate="1" pin="OUT"/>
+<wire x1="58.42" y1="45.72" x2="60.96" y2="45.72" width="0.1524" layer="91"/>
+<label x="63.5" y="45.72" size="1.778" layer="95" xref="yes"/>
+<pinref part="R1" gate="G$1" pin="2"/>
+<wire x1="60.96" y1="45.72" x2="63.5" y2="45.72" width="0.1524" layer="91"/>
+<wire x1="60.96" y1="43.18" x2="60.96" y2="45.72" width="0.1524" layer="91"/>
+</segment>
+<segment>
+<pinref part="X3" gate="-1" pin="KL"/>
+<wire x1="17.78" y1="53.34" x2="20.32" y2="53.34" width="0.1524" layer="91"/>
+<label x="20.32" y="53.34" size="1.778" layer="95" xref="yes"/>
+</segment>
+</net>
+<net name="N$1" class="0">
+<segment>
+<pinref part="R2" gate="G$1" pin="E"/>
+<pinref part="IC1" gate="1" pin="ADJ"/>
+<wire x1="50.8" y1="33.02" x2="50.8" y2="38.1" width="0.1524" layer="91"/>
+<pinref part="R1" gate="G$1" pin="1"/>
+<wire x1="50.8" y1="33.02" x2="60.96" y2="33.02" width="0.1524" layer="91"/>
+</segment>
+</net>
